Commit message: use positions instead of displacements for reconstruction

File: gym_pybullet_drones/assets/sphere2green.urdf (robot description, URDF)
Before this commit: robot urdf_robot, 1 links, 0 joints
Links:
- link baseLink: geometry collision sphere radius=0.5; visual mesh filename=sphere_smooth.obj scale=0.5 0.5 0.5
